File: Eagle/pro/revB/revB.sch (EAGLE design)
At the start: 13 parts, among them IC1 ATMEGA644A, Q1 20MHz

Commit message: new pcb with a 644
Parts:
- added C1, C10, C11, C12, C4, C5, C6, C7, C8, C9: 100nF, SparkFun:CAP0805
- added C13: 22pF, SparkFun:CAP0805
- added JP1: (no value), SparkFun-Connectors:M03PTH
- added JP2: M10", SparkFun-Connectors:M10"
- added JP3: (no value), SparkFun-Connectors:M07
- added LED1, LED2, LED3: (no value), SparkFun:LED1206
- added R1, R11, R12: 4.7K, SparkFun:RESISTOR1206
- added R13, R14, R15: 68, SparkFun:RESISTOR1206
- added R2, R3, R6: 100K, SparkFun:RESISTOR1206
- added R4, R5: 100k, SparkFun:RESISTOR1206
- added R7: 330K, SparkFun:RESISTOR1206
- added S1, S2, S3: (no value), SparkFun:TAC_SWITCHPTH
- added SV1: (no value), con-lstb:MA03-2
- added U$2: AUDIO-JACKPTH, SparkFun:AUDIO-JACKPTH
- added U$3, U$4: LM393, SparkFun:LM393
- added U$5: POTTRIM, SparkFun:POTTRIM
- added U1: MCP42XXX, SparkFun:MCP42XXX
- added U2: MCP1826S-3302E/DB, MCP1826S:MCP1826S-3302E/DB
- added X2: USB-MB-H, SparkFun:USB-MB-H
Connections:
- new net BIAS_LEFT: JP3.5, U$3G1.-IN, U$3G1.OUT, U1.A0
- new net BIAS_RIGHT: JP3.4, U$3G2.-IN, U$3G2.OUT, U1.A1
- new net D+: IC1.(PCINT10/INT2/AIN0)PB2
- new net D-: IC1.(PCINT11/OC0A/AIN1)PB3
- new net DEBUG_RX: IC1.(PCINT24/RXD0)PD0, JP1.3
- new net DEBUG_TX: IC1.(PCINT25/TXD0)PD1, JP1.2
- new net LCD_A0: IC1.(PCINT21/TDI)PC5, JP2.4, U$1.A0
- new net LCD_CS: IC1.(PCINT20/TDO)PC4, JP2.5, U$1./CS1
- new net LCD_RST: IC1.(PCINT19/TMS)PC3, JP2.6, U$1./RST
- new net LED1: IC1.(PCINT29/OC1A)PD5, LED1.A
- new net LED2: IC1.(PCINT30/OC2B/ICP)PD6, LED2.A
- new net LED3: IC1.(PCINT31/OC2A)PD7, LED3.A
- new net MISO: IC1.(PCINT14/MISO)PB6, JP2.2, SV1.1, U1.DO
- new net MOSI: IC1.(PCINT13/MOSI)PB5, JP2.3, SV1.4, U$1.SI, U1.DI
- new net N$10: C6.1, U$1.V3
- new net N$11: C7.1, U$1.V4
- new net N$12: C8.1, U$1.VOUT
- new net N$13: S1.3, S1.4, SV1.5
- new net N$15: C11.2, R2.1, R3.2, U$3G2.+IN
- new net N$16: C12.2, R4.1, R5.2, U$3G1.+IN
- new net N$17: C13.2, R7.1, U$4G2.+IN
- new net N$20: U2.VIN, X2.VBUS
- new net N$22: LED1.C, R13.2
- new net N$23: LED2.C, R14.2
- new net N$24: LED3.C, R15.2
- new net N$3: C9.2, U$1.C2-
- new net N$4: C9.1, U$1.C2+
- new net N$5: C10.2, U$1.C1+
- new net N$6: C10.1, U$1.C1-
- new net N$7: C1.1, U$1.V0
- new net N$8: C4.1, U$1.V1
- new net N$9: C5.1, U$1.V2
- new net POT_CS: IC1.(PCINT17/SDA)PC1, JP2.8, U1.CS
- new net POT_RST: IC1.(PCINT16/SCL)PC0, JP2.9, U1.RST
- new net POT_SHDW: IC1.(PCINT18/TCK)PC2, JP2.7, U1.SHTDWN
- new net RAW_LEFT: C12.1, JP3.3, U$2.5
- new net RAW_RIGHT: C11.1, JP3.2, U$2.2
- new net RESET: IC1.RESET, R1.1
- new net SCK: IC1.(PCINT15/SCK)PB7, JP2.1, SV1.3, U$1.SCL, U1.SCK
- new net SUM: R6.2, U$4G1.-IN, U1.W0, U1.W1
- new net SUMMED: JP3.6, R6.1, R7.2, U$4G1.OUT
- new net SW1: IC1.(PCINT27/INT1)PD3, R11.2, S2.1, S2.2
- new net SW2: IC1.(PCINT28/OC1B)PD4, R12.2, S3.1, S3.2
- new net TO_ADC: IC1.(PCINT0/ADC0)PA0, JP3.7, U$4G2.-IN, U$4G2.OUT
- new net USER_TRIM: IC1.(PCINT1/ADC1)PA1, U$5.S
- net GND: now also C1.2, C13.1, C4.2, C5.2, C6.2, C7.2, C8.2, JP1.1, JP2.10, JP3.1, R11.1, R12.1, R13.1, R14.1, R15.1, R3.1, R5.1, S1.1, S1.2, SV1.6, U$1.K, U$1.VSS, U$2.1, U$3G1.V-, U$4G1.+IN, U$4G1.V-, U$5.E, U1.GND, U2.GND_(TAB), U2.GND_(TAB)_2, X2.GND
- net VCC: now also R1.2, R2.2, R4.2, S2.3, S2.4, S3.3, S3.4, SV1.2, U$1.A, U$1.VDD, U$3G1.V+, U$4G1.V+, U$5.A, U1.VCC, U2.VOUT
